File: pcb/CC1TXUC.sch (KiCad schematic (older format))
At the start: 95 parts, among them J2 3.5 mm stereo, J3 I2C, J4 AVR-ISP-6, J5 UART, J6 GPS, J7 ADC, J8 +12VDC, J9 BNC, P3 TX Drive, P5 +3.3V, P6 +12V, P7 GND, P8 +5V, P9 VFO, Q10 IRLML9301, Q9 FDS86106, U2 74AC08, U3 ATMEGA328P, U4 VCC1-B3D-50M0000000, U5 AD9834, U6 LP2985-3.3, U7 LP2985-5, U8 OPA820IDBVT

Commit message: Update schematics for beta
Parts:
- C42: value 100n -> 10n
- D5: value BZV55-B15 -> BZV55-B33
- R43, R44, R45: value 33k -> 10k
- R61: value 2.2k -> 3.3k
- R62: value 51 -> 47
Other:
- note added: "All capacitors in pF unless specified"
- moved on the sheet: C72, C76, P9, R58, R59, R60, R61, R62, U8
Changed lines of the file:
@@
-EESchema Schematic File Version 2  date Wed 09 Jan 2013 07:00:57 PM PST
+EESchema Schematic File Version 2  date Thu 31 Jan 2013 03:10:17 PM PST
 LIBS:NT7S
 LIBS:power
@@
 Sheet 3 3
 Title "CC1 Transceiver"
-Date "10 jan 2013"
+Date "31 jan 2013"
 Rev "A"
 Comp "Etherkit"
@@
 P 4465 6820
 F 0 "D5" V 4260 6875 50  0000 C CNN
-F 1 "BZV55-B15" V 4180 6695 50  0000 C CNN
+F 1 "BZV55-B33" V 4180 6695 50  0000 C CNN
 	1    4465 6820
 	0    -1   -1   0
@@
 P 2350 3100
 F 0 "R45" H 2200 3205 50  0000 C CNN
-F 1 "33k" H 2195 3135 50  0000 C CNN
+F 1 "10k" H 2195 3135 50  0000 C CNN
 	1    2350 3100
 	1    0    0    -1
@@
 P 2150 3310
 F 0 "R44" V 1985 3275 50  0000 C CNN
-F 1 "33k" V 2055 3280 50  0000 C CNN
+F 1 "10k" V 2055 3280 50  0000 C CNN
 	1    2150 3310
 	0    1    1    0
@@
 P 1770 3310
 F 0 "R43" V 1610 3280 50  0000 C CNN
-F 1 "33k" V 1680 3275 50  0000 C CNN
+F 1 "10k" V 1680 3275 50  0000 C CNN
 	1    1770 3310
 	0    1    1    0
@@
 P 1015 3550
 F 0 "C42" V 1240 3565 50  0000 C CNN
-F 1 "100n" V 1155 3540 50  0000 C CNN
+F 1 "10n" V 1155 3540 50  0000 C CNN
 	1    1015 3550
 	0    -1   -1   0
@@
 L R R61
 U 1 1 50E38CB8
-P 9525 2140
-F 0 "R61" V 9355 2130 50  0000 C CNN
-F 1 "2.2k" V 9430 2140 50  0000 C CNN
-	1    9525 2140
+P 9350 2140
+F 0 "R61" V 9180 2130 50  0000 C CNN
+F 1 "3.3k" V 9255 2140 50  0000 C CNN
+	1    9350 2140
 	0    1    1    0
 $EndComp
@@
 L OPAMP-SOT23 U8
 U 1 1 50E38CC0
-P 9415 2595
-F 0 "U8" H 9325 2210 50  0000 L CNN
-F 1 "OPA820IDBVT" H 9325 2140 50  0000 L CNN
-	1    9415 2595
+P 9240 2595
+F 0 "U8" H 9150 2210 50  0000 L CNN
+F 1 "OPA820IDBVT" H 9150 2140 50  0000 L CNN
+	1    9240 2595
 	1    0    0    -1
 $EndComp
@@
 L R R59
 U 1 1 50E38CCD
-P 8875 2495
-F 0 "R59" V 8710 2490 50  0000 C CNN
-F 1 "220" V 8775 2485 50  0000 C CNN
-	1    8875 2495
+P 8700 2495
+F 0 "R59" V 8535 2490 50  0000 C CNN
+F 1 "220" V 8600 2485 50  0000 C CNN
+	1    8700 2495
 	0    1    1    0
 $EndComp
@@
 L GND #PWR0131
 U 1 1 50E38D0F
-P 9315 2875
-F 0 "#PWR0131" H 9315 2875 30  0001 C CNN
-F 1 "GND" H 9315 2805 30  0001 C CNN
-	1    9315 2875
+P 9140 2875
+F 0 "#PWR0131" H 9140 2875 30  0001 C CNN
+F 1 "GND" H 9140 2805 30  0001 C CNN
+	1    9140 2875
 	1    0    0    -1
 $EndComp
@@
 L R R58
 U 1 1 50E38D15
-P 8675 2695
-F 0 "R58" V 8790 2575 50  0000 C CNN
-F 1 "4.7k" V 8855 2580 50  0000 C CNN
-	1    8675 2695
+P 8500 2695
+F 0 "R58" V 8615 2575 50  0000 C CNN
+F 1 "4.7k" V 8680 2580 50  0000 C CNN
+	1    8500 2695
 	0    1    1    0
 $EndComp
@@
 L R R60
 U 1 1 50E38D25
-P 8875 2865
-F 0 "R60" H 8725 2810 50  0000 C CNN
-F 1 "4.7k" H 8730 2745 50  0000 C CNN
-	1    8875 2865
+P 8700 2865
+F 0 "R60" H 8550 2810 50  0000 C CNN
+F 1 "4.7k" H 8555 2745 50  0000 C CNN
+	1    8700 2865
 	1    0    0    -1
 $EndComp
@@
 L C C72
 U 1 1 50E38D2B
-P 9030 2855
-F 0 "C72" H 8900 2940 50  0000 C CNN
-F 1 "10n" H 8900 3005 50  0000 C CNN
-	1    9030 2855
+P 8855 2855
+F 0 "C72" H 8725 2940 50  0000 C CNN
+F 1 "10n" H 8725 3005 50  0000 C CNN
+	1    8855 2855
 	-1   0    0    1
 $EndComp
@@
 L R R62
 U 1 1 50E38DCE
-P 9815 2775
-F 0 "R62" H 9690 2810 50  0000 C CNN
-F 1 "51" H 9665 2745 50  0000 C CNN
-	1    9815 2775
-	1    0    0    -1
+P 9760 2595
+F 0 "R62" V 9925 2595 50  0000 C CNN
+F 1 "47" V 9855 2595 50  0000 C CNN
+	1    9760 2595
+	0    -1   -1   0
 $EndComp
 $Comp
 L C C76
 U 1 1 50E38DD4
-P 9975 2595
-F 0 "C76" V 10180 2590 50  0000 C CNN
-F 1 "10n" V 10115 2585 50  0000 C CNN
-	1    9975 2595
+P 10045 2595
+F 0 "C76" V 10250 2590 50  0000 C CNN
+F 1 "10n" V 10185 2585 50  0000 C CNN
+	1    10045 2595
 	0    -1   -1   0
-$EndComp
-$Comp
-L GND #PWR0132
-U 1 1 50E38FC7
-P 9815 2945
-F 0 "#PWR0132" H 9815 2945 30  0001 C CNN
-F 1 "GND" H 9815 2875 30  0001 C CNN
-	1    9815 2945
-	1    0    0    -1
 $EndComp
 $Comp
 L +5V #PWR0133
 U 1 1 50E3924D
-P 9315 2310
-F 0 "#PWR0133" H 9315 2400 20  0001 C CNN
-F 1 "+5V" H 9315 2400 30  0000 C CNN
-	1    9315 2310
+P 9140 2310
+F 0 "#PWR0133" H 9140 2400 20  0001 C CNN
+F 1 "+5V" H 9140 2400 30  0000 C CNN
+	1    9140 2310
 	1    0    0    -1
 $EndComp
@@
 L +5V #PWR0134
 U 1 1 50E392B3
-P 8525 2655
-F 0 "#PWR0134" H 8525 2745 20  0001 C CNN
-F 1 "+5V" H 8525 2745 30  0000 C CNN
-	1    8525 2655
-	1    0    0    -1
-$EndComp
-Text GLabel 10215 2595 2    40   Output ~ 0
+P 8350 2655
+F 0 "#PWR0134" H 8350 2745 20  0001 C CNN
+F 1 "+5V" H 8350 2745 30  0000 C CNN
+	1    8350 2655
+	1    0    0    -1
+$EndComp
+Text GLabel 10285 2595 2    40   Output ~ 0
 VFO
 Wire Wire Line
-	9315 2845 9315 2875
+	9140 2845 9140 2875
 $Comp
 L GND #PWR0135
 U 1 1 50E39697
-P 8875 3030
-F 0 "#PWR0135" H 8875 3030 30  0001 C CNN
-F 1 "GND" H 8875 2960 30  0001 C CNN
-	1    8875 3030
+P 8700 3030
+F 0 "#PWR0135" H 8700 3030 30  0001 C CNN
+F 1 "GND" H 8700 2960 30  0001 C CNN
+	1    8700 3030
 	1    0    0    -1
 $EndComp
@@
 L GND #PWR0136
 U 1 1 50E3969D
-P 9030 3030
-F 0 "#PWR0136" H 9030 3030 30  0001 C CNN
-F 1 "GND" H 9030 2960 30  0001 C CNN
-	1    9030 3030
-	1    0    0    -1
-$EndComp
-Wire Wire Line
-	9030 2955 9030 3030
-Wire Wire Line
-	8875 3015 8875 3030
-Wire Wire Line
-	10075 2595 10215 2595
-Wire Wire Line
-	9715 2595 9875 2595
-Wire Wire Line
-	9815 2140 9815 2625
-Connection ~ 9815 2595
-Wire Wire Line
-	9815 2925 9815 2945
-Wire Wire Line
-	8525 2655 8525 2695
-Wire Wire Line
-	8825 2695 9115 2695
-Wire Wire Line
-	9030 2755 9030 2695
-Connection ~ 9030 2695
-Wire Wire Line
-	8875 2715 8875 2695
-Connection ~ 8875 2695
-Wire Wire Line
-	9315 2310 9315 2345
-Wire Wire Line
-	9025 2495 9115 2495
-Wire Wire Line
-	9375 2140 9030 2140
-Wire Wire Line
-	9030 2140 9030 2495
-Connection ~ 9030 2495
-Wire Wire Line
-	9675 2140 9815 2140
-Wire Wire Line
-	8725 2495 8665 2495
-Wire Wire Line
-	8665 2495 8665 1850
-Wire Wire Line
-	8665 1850 9780 1850
+P 8855 3030
+F 0 "#PWR0136" H 8855 3030 30  0001 C CNN
+F 1 "GND" H 8855 2960 30  0001 C CNN
+	1    8855 3030
+	1    0    0    -1
+$EndComp
+Wire Wire Line
+	8855 2955 8855 3030
+Wire Wire Line
+	8700 3015 8700 3030
+Wire Wire Line
+	10145 2595 10285 2595
+Wire Wire Line
+	8350 2655 8350 2695
+Wire Wire Line
+	8650 2695 8940 2695
+Wire Wire Line
+	8855 2755 8855 2695
+Connection ~ 8855 2695
+Wire Wire Line
+	8700 2715 8700 2695
+Connection ~ 8700 2695
+Wire Wire Line
+	9140 2310 9140 2345
+Wire Wire Line
+	8850 2495 8940 2495
+Wire Wire Line
+	9200 2140 8855 2140
+Wire Wire Line
+	8855 2140 8855 2495
+Connection ~ 8855 2495
+Wire Wire Line
+	8550 2495 8490 2495
+Wire Wire Line
+	8490 2495 8490 1850
+Wire Wire Line
+	8490 1850 9780 1850
 Wire Wire Line
 	9780 1850 9780 1490
@@
 Text Notes 2265 3930 0    80   Italic 0
 Microcontroller
-Text Notes 7745 2740 0    80   Italic 0
+Text Notes 6955 2720 0    80   Italic 0
 DDS VFO
 $Comp
@@
 L CONN_1 P9
 U 1 1 50E3E182
-P 10330 2425
-F 0 "P9" H 10410 2425 40  0000 L CNN
-F 1 "VFO" H 10330 2480 30  0000 C CNN
-	1    10330 2425
-	1    0    0    -1
-$EndComp
-Wire Wire Line
-	10180 2425 10110 2425
-Wire Wire Line
-	10110 2425 10110 2595
-Connection ~ 10110 2595
+P 10400 2425
+F 0 "P9" H 10360 2530 40  0000 L CNN
+F 1 "VFO" H 10400 2480 30  0000 C CNN
+	1    10400 2425
+	1    0    0    -1
+$EndComp
+Wire Wire Line
+	10250 2425 10180 2425
+Wire Wire Line
+	10180 2425 10180 2595
+Connection ~ 10180 2595
 $Comp
 L CONN_1 P7
@@
 Wire Wire Line
 	1545 7755 1545 7735
+Wire Wire Line
+	9945 2595 9910 2595
+Wire Wire Line
+	9610 2595 9540 2595
+Wire Wire Line
+	9500 2140 9570 2140
+Wire Wire Line
+	9570 2140 9570 2595
+Connection ~ 9570 2595
+Text Notes 8740 6960 0    60   ~ 0
+All capacitors in pF unless specified
 $EndSCHEMATC
